Commit message: add rviz mobiel

File: exbotxi_description/urdf/irobot_create.urdf.xacro (robot description, xacro)
@@ -73,5 +73,5 @@
       </collision>
     </link>
-    <joint name="base_l_wheel_joint" type="continuous">
+    <joint name="base_l_wheel_joint" type="fixed">
       <origin xyz="0 0.13 0.015" rpy="0 0 0"/>
       <parent link="base_link"/>
@@ -99,5 +99,5 @@
       </collision>
     </link>
-    <joint name="base_r_wheel_joint" type="continuous">
+    <joint name="base_r_wheel_joint" type="fixed">
       <origin xyz="0 -0.13 0.015" rpy="0 0 0"/>
       <parent link="base_link"/>
