Commit message: add laser property

File: exbotxi_description/urdf/create_frame.urdf.xacro (robot description, xacro)
@@ -89,5 +89,5 @@
   </link>
   <joint name="laser_joint" type="fixed">
-    <origin xyz="0 0 0.06" rpy="0 0 0"/>
+    <origin xyz="${laser_px} ${laser_py} ${laser_pz+0.06}" rpy="0 0 0"/>
     <parent link="plate0_link"/>
     <child link="laser_link"/>

File: exbotxi_description/urdf/exbotxi_create.urdf.xacro (robot description, xacro)
@@ -4,4 +4,5 @@
   <xacro:property name="M_PI" value="3.1415926535897931" />
   <xacro:property name="H_PI" value="1.5707963" />
+  <xacro:include filename="$(find exbotxi_description)/urdf/properties.urdf.xacro" />
   <xacro:include filename="$(find exbotxi_description)/urdf/create_base.urdf.xacro"/>
   <xacro:include filename="$(find exbotxi_description)/urdf/create_frame.urdf.xacro"/>

File: exbotxi_description/urdf/exbotxi_kobuki.urdf.xacro (robot description, xacro)
@@ -6,4 +6,5 @@
   <xacro:include filename="$(find kobuki_description)/urdf/kobuki.urdf.xacro" />
   <kobuki/>
+  <xacro:include filename="$(find exbotxi_description)/urdf/properties.urdf.xacro" />
   <xacro:include filename="$(find exbotxi_description)/urdf/kobuki_frame.urdf.xacro"/>
   <xacro:include filename="$(find exbotxi_description)/urdf/xtion_pro.urdf.xacro"/>

File: exbotxi_description/urdf/kobuki_frame.urdf.xacro (robot description, xacro)
@@ -89,5 +89,5 @@
   </link>
   <joint name="laser_joint" type="fixed">
-    <origin xyz="0 0 0.06" rpy="0 0 0"/>
+    <origin xyz="${laser_px} ${laser_py} ${laser_pz+0.06}" rpy="0 0 0"/>
     <parent link="plate0_link"/>
     <child link="laser_link"/>
